File: Vector_XY_Driver.brd (EAGLE design)
At the start: 148.6 x 90.2 mm, 90 parts, among them IC1 LT 1227, IC2 LT 1227, IC3 LM393N, Q1 TIP142, Q2 TIP147, Q3 TIP142, Q4 TIP147, T2 BD243, T3 BD243, T4 BD244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

Commit message: Updated README
Parts:
- moved C5 4.49 mm to (76.2, 40.6), turned to 90 degrees
- moved D1 2.29 mm to (62.2, 17.8)
- moved C4 2.29 mm to (59.7, 21.0)
- moved R9 2.29 mm to (63.5, 26.7)
- moved R11 2.29 mm to (63.5, 24.1)
- moved IC3 1.91 mm to (66.0, 35.6)
- moved R12 1.91 mm to (72.4, 34.3)
- moved R10 1.90 mm to (59.7, 34.9)
Routing:
- net GND: track 347.2 -> 335.4 mm
- net N$43: track 40.8 -> 41.6 mm
- net N$40: track 33.0 -> 33.8 mm
- net V+: track 241.7 -> 241.0 mm
- net N$27: track 6.98 -> 6.35 mm
- net N$36: track 22.6 -> 22.1 mm
